File: Hardware/HiHat.kicad_pcb (KiCad board)
At the start: 2 copper layers, 63.5 x 105.4 mm, 47 parts, among them J1 CH trig in, J2 OH trig in, J3 IDC power connector, J4 Output, Q1 BC549, Q2 BC549, Q3 BC549, Q4 BC549, U1 TL074

Commit message: PCB routing
Parts:
- removed J4: Output, Connector_PinHeader_2.54mm:PinHeader_1x02_P2.54mm_Vertical
- removed MH: MountingHole_3.2mm_M3_DIN965_Pad, MountingHole:MountingHole_3.2mm_M3_DIN965_Pad
- J1: value CH trig in -> Inputs; footprint Connector_PinHeader_2.54mm:PinHeader_1x02_P2.54mm_Vertical -> Connector_JST:JST_EH_B3B-EH-A_1x03_P2.50mm_Vertical
- J2: value OH trig in -> Output; footprint Connector_PinHeader_2.54mm:PinHeader_1x02_P2.54mm_Vertical -> Connector_JST:JST_EH_B2B-EH-A_1x02_P2.50mm_Vertical
- moved C10 126.2 mm to (100.3, 121.9), turned to 90 degrees
- moved J1 116.0 mm to (85.1, 114.3), turned to 270 degrees
- moved J2 115.7 mm to (109.2, 137.2), turned to 90 degrees
- moved C6 108.5 mm to (92.7, 76.2), turned to 90 degrees
- moved D4 105.7 mm to (108.0, 113.0), turned to 180 degrees
- moved R9 103.5 mm to (87.6, 86.4), turned to 90 degrees
- moved C5 101.9 mm to (94.0, 82.5), turned to 180 degrees
- moved R14 98.3 mm to (88.9, 121.9), turned to 90 degrees
- moved R12 97.2 mm to (78.7, 127.0)
- moved R13 96.4 mm to (88.9, 124.5), turned to 180 degrees
- moved C7 85.9 mm to (106.7, 105.4), turned to 180 degrees
- moved D3 85.8 mm to (97.8, 76.2)
- moved C11 84.6 mm to (94.0, 121.9), turned to 90 degrees
- moved R11 79.2 mm to (105.4, 125.7), turned to 90 degrees
- moved D2 78.1 mm to (97.8, 73.7)
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Connections:
- C10 pad 2: Net-(C10-Pad2) -> OHtrig
- C11 pad 2: Net-(C11-Pad2) -> CHtrig
- J1 pad 1: GND -> CHtrig
- J1 pad 2: Net-(C11-Pad2) -> GND
- J2 pad 1: GND -> Net-(J2-Pad1)
- J2 pad 2: Net-(C10-Pad2) -> GND
- R15 pad 1: Net-(J4-Pad1) -> Net-(J2-Pad1)
Routing:
- net Net-(C5-Pad1): track 0.00 -> 66.6 mm
- net Net-(C6-Pad1): track 0.00 -> 58.4 mm
- net env: track 0.00 -> 45.1 mm
- net Net-(C5-Pad2): track 0.00 -> 40.7 mm
- net Net-(C7-Pad1): track 0.00 -> 38.5 mm
- net Net-(R12-Pad2): track 0.00 -> 22.9 mm, vias 0 -> 2
- net Net-(C7-Pad2): track 0.00 -> 21.4 mm
- net Net-(C8-Pad1): track 0.00 -> 21.4 mm
- net OHtrig: track 0.00 -> 16.3 mm
- net Net-(C10-Pad1): track 0.00 -> 15.0 mm
- net Net-(C11-Pad1): track 0.00 -> 14.0 mm
- net Net-(Q4-Pad1): track 0.00 -> 12.5 mm
- net CHtrig: track 0.00 -> 10.9 mm
- net Net-(R8-Pad2): track 0.00 -> 10.5 mm
- net Net-(D1-Pad1): track 0.00 -> 9.94 mm
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
Commit message: PCB routing
Parts:
- added REF**: MountingHole_3.2mm_M3_DIN965_Pad, MountingHole:MountingHole_3.2mm_M3_DIN965_Pad, F.Cu at (111.8, 166.4)
- added REF**: MountingHole_3.2mm_M3_DIN965_Pad, MountingHole:MountingHole_3.2mm_M3_DIN965_Pad, F.Cu at (76.2, 72.4)
- added REF**: MountingHole_3.2mm_M3_DIN965_Pad, MountingHole:MountingHole_3.2mm_M3_DIN965_Pad, F.Cu at (76.2, 166.4)
- moved C12 38.9 mm to (109.2, 160.0), turned to 90 degrees
- moved J3 26.9 mm to (90.2, 165.1), turned to 90 degrees
- moved C7 19.2 mm to (104.1, 86.4), turned to 0 degrees
- moved C13 18.0 mm to (81.3, 161.3)
- moved D5 8.98 mm to (106.7, 91.4), turned to 180 degrees
- moved R15 6.48 mm to (108.0, 135.9)
- moved C11 6.48 mm to (92.7, 115.6)
- moved C9 6.48 mm to (83.8, 125.7)
- moved R14 6.48 mm to (87.6, 115.6)
- moved C10 6.48 mm to (99.1, 115.6)
- moved U1 6.48 mm to (102.9, 124.5)
- moved C4 6.48 mm to (87.6, 140.3)
- moved J1 6.48 mm to (83.8, 108.0)
- moved R13 6.48 mm to (87.6, 118.1)
- moved J2 6.48 mm to (108.0, 130.8)
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Routing:
- net +12V: track 66.9 -> 100.8 mm, vias 2 -> 0
- net -12V: track 36.9 -> 69.2 mm, vias 0 -> 2
- net Net-(C7-Pad2): track 21.4 -> 7.64 mm
- net Net-(C5-Pad2): track 40.7 -> 29.0 mm, vias 0 -> 2
- net Net-(C5-Pad1): track 66.6 -> 58.4 mm
- net Net-(C7-Pad1): track 38.5 -> 46.1 mm
- net Net-(C6-Pad1): track 58.4 -> 52.6 mm
- net Net-(C8-Pad1): track 21.4 -> 16.1 mm
- net Net-(Q4-Pad2): track 4.86 -> 9.94 mm
- net Net-(Q4-Pad1): track 12.5 -> 8.67 mm
- net Net-(R8-Pad2): track 10.5 -> 9.20 mm
- net Net-(R15-Pad2): track 20.4 -> 21.4 mm
- net CHtrig: track 10.9 -> 9.98 mm
- net Net-(C1-Pad1): track 8.89 -> 9.42 mm
- net Net-(C10-Pad1): track 15.0 -> 15.5 mm
Other:
- board size 63.5 x 105.4 mm -> 40.6 x 99.1 mm
- board text added: "03 2021"
- board text added: "Simple hihat"
